File: hardware/r0.1a/M17-SmartMic.kicad_pcb (KiCad board)
At the start: 4 copper layers, 84.9 x 89.9 mm, 154 parts, among them J1 STLink, J2 USB_C, J3 OLED, J4 Kenwood-2.5, J5 Kenwood-3.5, J6 MBIAS, J7 Radio, Q1 IRLML2060, SW1 Button Up, SW2 Button Down, SW3 Reset, SW4 Button Green, SW5 Button Left, SW6 Button Red, SW7 Button Right, U1 STM32F407VETx, U2 LM1117-3.3, U3 USBLC6-2, U5 LM386, U6 LMV341, U7 MCP6002-xSN, U8 MCP6002-xSN, X1 12 MHz TCXO, Y1 8 MHz

Commit message: Added RTC
Changed lines of the file:
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@@
       (layerselection 0x00010fc_ffffffff)
       (disableapertmacros false)
-      (usegerberextensions false)
+      (usegerberextensions true)
       (usegerberattributes true)
       (usegerberadvancedattributes true)
@@
       (outputformat 1)
       (mirror false)
-      (drillshape 1)
+      (drillshape 0)
       (scaleselection 1)
-      (outputdirectory "")
+      (outputdirectory "gerber/")
     )
   )
@@
     (fp_line (start -3 -0.8) (end -3 1.6) (layer "F.Fab") (width 0.1))
     (fp_line (start -3 1.6) (end 3 1.6) (layer "F.Fab") (width 0.1))
-    (pad "1" smd roundrect locked (at -2.4625 0 270) (size 2.075 2.35) (layers "F.Cu" "F.Paste" "F.Mask") (roundrect_rratio 0.120482)
+    (pad "1" smd roundrect locked (at -2.4625 0 270) (size 2.075 2.35) (layers "F.Cu" "F.Paste" "F.Mask") (roundrect_rratio 0.1204819277)
       (net 32 "Net-(C52-Pad1)") (pintype "passive"))
-    (pad "2" smd roundrect locked (at 2.4625 0 270) (size 2.075 2.35) (layers "F.Cu" "F.Paste" "F.Mask") (roundrect_rratio 0.120482)
+    (pad "2" smd roundrect locked (at 2.4625 0 270) (size 2.075 2.35) (layers "F.Cu" "F.Paste" "F.Mask") (roundrect_rratio 0.1204819277)
       (net 2 "GND") (pintype "passive"))
     (model "${KISYS3DMOD}/Capacitor_Tantalum_SMD.3dshapes/CP_EIA-6032-28_Kemet-C.wrl"
@@
     (fp_line (start -1.2 -0.8) (end -1.6 -0.4) (layer "F.Fab") (width 0.1))
     (fp_line (start -1.6 0.8) (end 1.6 0.8) (layer "F.Fab") (width 0.1))
-    (pad "1" smd roundrect locked (at -1.35 0 90) (size 1.4 1.35) (layers "F.Cu" "F.Paste" "F.Mask") (roundrect_rratio 0.185185)
+    (pad "1" smd roundrect locked (at -1.35 0 90) (size 1.4 1.35) (layers "F.Cu" "F.Paste" "F.Mask") (roundrect_rratio 0.1851851852)
       (net 9 "+5V") (pintype "passive"))
-    (pad "2" smd roundrect locked (at 1.35 0 90) (size 1.4 1.35) (layers "F.Cu" "F.Paste" "F.Mask") (roundrect_rratio 0.185185)
+    (pad "2" smd roundrect locked (at 1.35 0 90) (size 1.4 1.35) (layers "F.Cu" "F.Paste" "F.Mask") (roundrect_rratio 0.1851851852)
       (net 2 "GND") (pintype "passive"))
     (model "${KISYS3DMOD}/Capacitor_Tantalum_SMD.3dshapes/CP_EIA-3216-18_Kemet-A.wrl"
@@
     (fp_line (start -3 1.6) (end 3 1.6) (layer "F.Fab") (width 0.1))
     (fp_line (start 3 -1.6) (end -2.2 -1.6) (layer "F.Fab") (width 0.1))
-    (pad "1" smd roundrect locked (at -2.4625 0 270) (size 2.075 2.35) (layers "F.Cu" "F.Paste" "F.Mask") (roundrect_rratio 0.120482)
+    (pad "1" smd roundrect locked (at -2.4625 0 270) (size 2.075 2.35) (layers "F.Cu" "F.Paste" "F.Mask") (roundrect_rratio 0.1204819277)
       (net 28 "Net-(C49-Pad1)") (pintype "passive"))
-    (pad "2" smd roundrect locked (at 2.4625 0 270) (size 2.075 2.35) (layers "F.Cu" "F.Paste" "F.Mask") (roundrect_rratio 0.120482)
+    (pad "2" smd roundrect locked (at 2.4625 0 270) (size 2.075 2.35) (layers "F.Cu" "F.Paste" "F.Mask") (roundrect_rratio 0.1204819277)
       (net 29 "Net-(C49-Pad2)") (pintype "passive"))
     (model "${KISYS3DMOD}/Capacitor_Tantalum_SMD.3dshapes/CP_EIA-6032-28_Kemet-C.wrl"
@@
     (fp_line (start 3 -1.6) (end -2.2 -1.6) (layer "F.Fab") (width 0.1))
     (fp_line (start -3 -0.8) (end -3 1.6) (layer "F.Fab") (width 0.1))
-    (pad "1" smd roundrect locked (at -2.4625 0 90) (size 2.075 2.35) (layers "F.Cu" "F.Paste" "F.Mask") (roundrect_rratio 0.120482)
+    (pad "1" smd roundrect locked (at -2.4625 0 90) (size 2.075 2.35) (layers "F.Cu" "F.Paste" "F.Mask") (roundrect_rratio 0.1204819277)
       (net 34 "Net-(C53-Pad2)") (pintype "passive"))
-    (pad "2" smd roundrect locked (at 2.4625 0 90) (size 2.075 2.35) (layers "F.Cu" "F.Paste" "F.Mask") (roundrect_rratio 0.120482)
+    (pad "2" smd roundrect locked (at 2.4625 0 90) (size 2.075 2.35) (layers "F.Cu" "F.Paste" "F.Mask") (roundrect_rratio 0.1204819277)
       (net 40 "Net-(C59-Pad2)") (pintype "passive"))
     (model "${KISYS3DMOD}/Capacitor_Tantalum_SMD.3dshapes/CP_EIA-6032-28_Kemet-C.wrl"
@@
     (fp_line (start 3 -1.6) (end -2.2 -1.6) (layer "F.Fab") (width 0.1))
     (fp_line (start -3 1.6) (end 3 1.6) (layer "F.Fab") (width 0.1))
-    (pad "1" smd roundrect locked (at -2.4625 0 270) (size 2.075 2.35) (layers "F.Cu" "F.Paste" "F.Mask") (roundrect_rratio 0.120482)
+    (pad "1" smd roundrect locked (at -2.4625 0 270) (size 2.075 2.35) (layers "F.Cu" "F.Paste" "F.Mask") (roundrect_rratio 0.1204819277)
       (net 30 "Net-(C50-Pad1)") (pintype "passive"))
-    (pad "2" smd roundrect locked (at 2.4625 0 270) (size 2.075 2.35) (layers "F.Cu" "F.Paste" "F.Mask") (roundrect_rratio 0.120482)
+    (pad "2" smd roundrect locked (at 2.4625 0 270) (size 2.075 2.35) (layers "F.Cu" "F.Paste" "F.Mask") (roundrect_rratio 0.1204819277)
       (net 2 "GND") (pintype "passive"))
     (model "${KISYS3DMOD}/Capacitor_Tantalum_SMD.3dshapes/CP_EIA-6032-28_Kemet-C.wrl"
