File: hardware/r0.1e/M17-SmartMic.kicad_pcb (KiCad board)
At the start: 4 copper layers, 84.9 x 89.9 mm, 184 parts, among them IC1 LM4861M, J1 Kenwood-2.5, J10 UART, J11 Radio_Opt, J12 Speaker, J2 USB_C, J3 OLED, J4 CAT_TX, J5 Kenwood-3.5, J6 CAT_TX, J7 Radio, J8 +12V, J9 STLink, Q1 IRLML2060, Q2 BSS138, Q3 BSS138, Q4 IRLML2244, Q5 MMBT3904, SW1 Button Up, SW2 Button Down, SW3 Reset, SW4 Button Escape, SW5 Button Left, SW6 Button Enter, SW7 Button Right, SW8 Button Power, U1 MAX9814, U10 STM32F405RGTx, U11 TPS7A2033, U2 TP6841S6, U3 USBLC6-2, U6 MCP6002, U7 MCP6002, X1 12 MHz TCXO, Y1 8 MHz

Commit message: Fix KC1AWV original fixes
Fix schematic and PCB layout. Populate R53 with 0R and update BOM to include R31 change
Parts:
- R31: value 22k -> 1k8
- R53: value 2k7 -> 0
Changed lines of the file:
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@@
     (descr "Resistor SMD 0603 (Metric 1608), reflow soldering")
     (tags "resistor 0603")
-    (property "MPN" "Generic R/22k/0603")
+    (property "MPN" "Generic R/1k8/0603")
     (property "Sheetfile" "Audio.kicad_sch")
     (property "Sheetname" "Audio & Filter")
@@
         (effects (font (size 0.635 0.635) (thickness 0.1)))
     )
-    (fp_text value "22k" (at 0 1.25) (layer "F.Fab")
+    (fp_text value "1k8" (at 0 1.25) (layer "F.Fab")
         (effects (font (size 0.635 0.635) (thickness 0.1)))
     )
@@
     (property "Sheetfile" "Microcontroller.kicad_sch")
     (property "Sheetname" "Microcontroller")
+    (property "dnp" "")
     (property "ki_description" "Resistor")
     (attr smd exclude_from_pos_files)
@@
     (descr "SOT, 3 Pin (https://www.jedec.org/system/files/docs/to-236h.pdf variant AB), generated with kicad-footprint-generator ipc_gullwing_generator.py")
     (tags "SOT TO_SOT_SMD")
-    (property "LCSC Part #" "C2912548")
+    (property "LCSC Part #" "C400505")
     (property "MPN" "BSS138P,215")
     (property "Sheetfile" "Audio.kicad_sch")
@@
     (descr "SOT, 3 Pin (https://www.jedec.org/system/files/docs/to-236h.pdf variant AB), generated with kicad-footprint-generator ipc_gullwing_generator.py")
     (tags "SOT TO_SOT_SMD")
-    (property "LCSC Part #" "C2912548")
+    (property "LCSC Part #" "C400505")
     (property "MPN" "BSS138P,215")
     (property "Sheetfile" "Audio.kicad_sch")
@@
     (descr "C&K Components, PTS 810 Series, Microminiature SMT Top Actuated, http://www.ckswitches.com/media/1476/pts810.pdf")
     (tags "SPST Button Switch")
-    (property "LCSC Part #" "C589193")
-    (property "MPN" "ST-1185SE")
+    (property "LCSC Part #" "C221895")
+    (property "MPN" "PTS810SJG250SMTRLFS")
     (property "Sheetfile" "Microcontroller.kicad_sch")
     (property "Sheetname" "Microcontroller")
@@
     (property "Sheetname" "Microcontroller")
     (property "ki_description" "Resistor")
-    (attr smd exclude_from_pos_files)
+    (attr smd)
     (fp_text reference "R53" (at 0 -1.25 90) (layer "F.Fab")
         (effects (font (size 0.635 0.635) (thickness 0.1)))
     )
-    (fp_text value "2k7" (at 0 1.25 90) (layer "F.Fab")
+    (fp_text value "0" (at 0 1.25 90) (layer "F.Fab")
         (effects (font (size 0.635 0.635) (thickness 0.1)))
     )
