File: hardware/Audio.kicad_sch (KiCad schematic)
At the start: 48 parts, among them IC1 LM4991xx, J4 CAT_TX, J6 CAT_TX, Q1 IRLML2060, Q2 BSS138, Q3 BSS138, U1 MAX9814, U201 MCP6002

Commit message: Updated various MPNs
Parts:
- C201: MPN (none) -> Generic C/10nF/C0G/25V/0603
- U201: LCSC Part # (none) -> C116706; MPN (none) -> MCP6002-I/SN
Changed lines of the file:
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@@
+      (effects (font (size 1.27 1.27)) hide)
+    )
+    (property "MPN" "MCP6002-I/SN" (at 83.82 44.45 0)
+      (effects (font (size 1.27 1.27)) hide)
+    )
+    (property "LCSC Part #" "C116706" (at 83.82 44.45 0)
       (effects (font (size 1.27 1.27)) hide)
     )
@@
       (effects (font (size 1.27 1.27)) hide)
     )
+    (property "MPN" "Generic C/10nF/C0G/25V/0603" (at 75.565 31.115 0)
+      (effects (font (size 1.27 1.27)) hide)
+    )
     (pin "1")
     (pin "2")
@@
     )
     (property "Datasheet" "http://ww1.microchip.com/downloads/en/DeviceDoc/21314g.pdf" (at 76.835 74.295 0)
+      (effects (font (size 1.27 1.27)) hide)
+    )
+    (property "MPN" "MCP6002-I/SN" (at 76.835 74.295 0)
+      (effects (font (size 1.27 1.27)) hide)
+    )
+    (property "LCSC Part #" "C116706" (at 76.835 74.295 0)
       (effects (font (size 1.27 1.27)) hide)
     )
@@
       (effects (font (size 1.27 1.27)) hide)
     )
+    (property "MPN" "MCP6002-I/SN" (at 52.07 72.39 0)
+      (effects (font (size 1.27 1.27)) hide)
+    )
+    (property "LCSC Part #" "C116706" (at 52.07 72.39 0)
+      (effects (font (size 1.27 1.27)) hide)
+    )
