File: hardware/mainboard/baseband.kicad_sch (KiCad schematic)
At the start: 36 parts, among them U501 MCP4551-103, U502 MCP4551-103, U503 MCP6002, U504 MCP6002

Commit message: Mainboard Rev 0.99b
Parts:
- C501, C502, C513, C514: MPN Generic C/100nF/C0G/25V/0603 -> Generic C/100nF/X7R/50V/0603
- RV501, RV502: LCSC Part # C81348 -> C465012
Changed lines of the file:
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@@
 	(title_block
 		(title "Module17")
-		(date "2023-12-06")
-		(rev "Rev 0.99")
+		(date "2024-04-25")
+		(rev "Rev 0.99b")
 		(company "M17Project")
 		(comment 1 "Morgan ON4MOD")
@@
 			)
 		)
-		(property "MPN" "Generic C/100nF/C0G/25V/0603"
+		(property "MPN" "Generic C/100nF/X7R/50V/0603"
 			(at 206.375 39.37 0)
 			(effects
@@
 			)
 		)
-		(property "LCSC Part #" "C81348"
+		(property "LCSC Part #" "C465012"
 			(at 120.65 83.185 0)
 			(effects
@@
 			)
 		)
-		(property "Datasheet" "~"
+		(property "Datasheet" ""
 			(at 53.975 161.29 0)
 			(effects
@@
 			)
 		)
-		(property "MPN" "Generic C/100nF/C0G/25V/0603"
+		(property "MPN" "Generic C/100nF/X7R/50V/0603"
 			(at 53.975 161.29 0)
 			(effects
@@
 			)
 		)
-		(property "LCSC Part #" "C81348"
+		(property "LCSC Part #" "C465012"
 			(at 102.235 167.64 0)
 			(effects
@@
 			)
 		)
-		(property "MPN" "Generic C/100nF/C0G/25V/0603"
+		(property "MPN" "Generic C/100nF/X7R/50V/0603"
 			(at 215.9 129.54 0)
 			(effects
@@
 			)
 		)
-		(property "Datasheet" "~"
+		(property "Datasheet" ""
 			(at 74.295 76.835 0)
 			(effects
@@
 			)
 		)
-		(property "MPN" "Generic C/100nF/C0G/25V/0603"
+		(property "MPN" "Generic C/100nF/X7R/50V/0603"
 			(at 74.295 76.835 0)
 			(effects

Commit message: Updated Mainboard PCB to revision 1.0
Other:
- company: M17Project -> M17 Project
Changed lines of the file:
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@@
 	(title_block
 		(title "Module17")
-		(date "2024-04-25")
-		(rev "Rev 0.99b")
-		(company "M17Project")
-		(comment 1 "Morgan ON4MOD")
+		(date "2024-06-19")
+		(rev "Rev 1.0")
+		(company "M17 Project")
+		(comment 1 "Morgan - ON4MOD")
 		(comment 2 "Mathis - DB9MAT")
 		(comment 3 "Wojciech - SP5WWP")
