File: hardware/mainboard/connectors.kicad_sch (KiCad schematic)
At the start: 25 parts, among them J401 Radio, J402 USB_C, J403 Radio_Opt, J404 Kenwood-3.5, J405 Kenwood-2.5, J406 2.54mm Header 7p, J407 KH-RJ45-58-8P8C, J408 STLink, J409 UART, J410 Speaker, J411 +12V, J412 Hirose FH12-26S-0.5SH(55), J413 Molex 532610271, U401 USBLC6-2SC6

Commit message: Mainboard Rev 0.99b
Parts:
- C401: MPN Generic C/100nF/C0G/25V/0603 -> Generic C/100nF/X7R/50V/0603
- J401: footprint Connector_Dsub:DSUB-9_Female_Horizontal_P2.77x2.84mm_EdgePinOffset4.94mm_Housed_MountingHolesOffset7.48mm -> Connector_Dsub:DSUB-9_Female_Horizontal_P2.77x2.84mm_EdgePinOffset7.70mm_Housed_MountingHolesOffset9.12mm
- J412: now fitted
Changed lines of the file:
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@@
 	(title_block
 		(title "Module17")
-		(date "2023-12-06")
-		(rev "Rev 0.99")
+		(date "2024-04-25")
+		(rev "Rev 0.99b")
 		(company "M17Project")
 		(comment 1 "Morgan ON4MOD")
@@
 		(in_bom yes)
 		(on_board yes)
-		(dnp yes)
+		(dnp no)
 		(fields_autoplaced yes)
 		(property "Reference" "J412"
@@
 			)
 		)
-		(property "MPN" "Generic C/100nF/C0G/25V/0603"
+		(property "MPN" "Generic C/100nF/X7R/50V/0603"
 			(at 53.34 158.75 0)
 			(effects
@@
 			)
 		)
-		(property "Footprint" "Connector_Dsub:DSUB-9_Female_Horizontal_P2.77x2.84mm_EdgePinOffset4.94mm_Housed_MountingHolesOffset7.48mm"
+		(property "Footprint" "Connector_Dsub:DSUB-9_Female_Horizontal_P2.77x2.84mm_EdgePinOffset7.70mm_Housed_MountingHolesOffset9.12mm"
 			(at 33.02 39.37 0)
 			(effects

Commit message: Updated Mainboard PCB to revision 1.0
Other:
- company: M17Project -> M17 Project
Changed lines of the file:
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@@
 	(title_block
 		(title "Module17")
-		(date "2024-04-25")
-		(rev "Rev 0.99b")
-		(company "M17Project")
-		(comment 1 "Morgan ON4MOD")
+		(date "2024-06-19")
+		(rev "Rev 1.0")
+		(company "M17 Project")
+		(comment 1 "Morgan - ON4MOD")
 		(comment 2 "Mathis - DB9MAT")
 		(comment 3 "Wojciech - SP5WWP")
