File: hardware/mainboard/mcu_power.kicad_sch (KiCad schematic)
At the start: 87 parts, among them Q201 MMBT3904, Q202 IRLML2244, SW201 Tactile switch, SW202 Tactile switch, SW203 Tactile switch, SW204 Tactile switch, SW205 Tactile switch, SW206 Tactile switch, SW207 Tactile switch, SW208 Tactile switch, U201 STM32F405RGTx, U202 TPS7A2033, U203 TP6841S6, Y201 8 MHz

Commit message: Mainboard Rev 0.99b
Parts:
- added R233: 0, Resistor_SMD:R_0603_1608Metric, symbol Device:R
- C201, C214, C219, C221, C227: MPN Generic C/10nF/C0G/25V/0603 -> Generic C/10nF/X7R/25V/0603
- C204, C205: MPN Generic C/2.2uF/C0G/25V/0603 -> Generic C/2.2uF/X5R/25V/0603
- C207: MPN Generic C/10uF/C0G/25V/1210 -> Generic C/10uF/X7R/25V/1210
- C208, C209, C210, C213, C215, C216, C217, C220, C225, C226: MPN Generic C/100nF/C0G/25V/0603 -> Generic C/100nF/X7R/50V/0603
- C211, C218, C222, C224: MPN Generic C/1uF/C0G/25V/0603 -> Generic C/1uF/X7R/25V/0603
- JP201: now not fitted
Connections:
- net +5V: now also R233.1
- net at C223.1, JP201.1 (A), L202.1: now also R233.2
Other:
- moved on the sheet: C223
Changed lines of the file:
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@@
 	(title_block
 		(title "Module17")
-		(date "2023-12-06")
-		(rev "Rev 0.99")
+		(date "2024-04-25")
+		(rev "Rev 0.99b")
 		(company "M17Project")
 		(comment 1 "Morgan ON4MOD")
@@
 	)
 	(junction
+		(at 198.755 146.05)
+		(diameter 0)
+		(color 0 0 0 0)
+	)
+	(junction
 		(at 146.685 151.13)
 		(diameter 0)
@@
 	)
 	(junction
+		(at 187.325 146.05)
+		(diameter 0)
+		(color 0 0 0 0)
+	)
+	(junction
 		(at 273.685 147.32)
 		(diameter 0)
@@
 	(wire
 		(pts
+			(xy 198.755 146.05) (xy 198.755 149.225)
+		)
+		(stroke
+			(width 0)
+			(type default)
+		)
+	)
+	(wire
+		(pts
 			(xy 106.045 99.695) (xy 108.585 99.695)
 		)
@@
 	(wire
 		(pts
-			(xy 182.245 146.05) (xy 187.96 146.05)
+			(xy 182.245 146.05) (xy 187.325 146.05)
 		)
 		(stroke
@@
 	(wire
 		(pts
-			(xy 182.245 146.05) (xy 182.245 148.59)
+			(xy 182.245 146.05) (xy 182.245 154.305)
 		)
 		(stroke
@@
 	(wire
 		(pts
+			(xy 196.85 149.225) (xy 198.755 149.225)
+		)
+		(stroke
+			(width 0)
+			(type default)
+		)
+	)
+	(wire
+		(pts
 			(xy 137.795 79.375) (xy 137.795 80.645)
 		)
@@
 	(wire
 		(pts
+			(xy 187.325 146.05) (xy 187.96 146.05)
+		)
+		(stroke
+			(width 0)
+			(type solid)
+		)
+	)
+	(wire
+		(pts
 			(xy 146.685 160.02) (xy 146.685 162.56)
 		)
@@
 	(wire
 		(pts
+			(xy 187.325 146.05) (xy 187.325 149.225)
+		)
+		(stroke
+			(width 0)
+			(type default)
+		)
+	)
+	(wire
+		(pts
 			(xy 159.385 154.94) (xy 159.385 158.75)
 		)
@@
 	(wire
 		(pts
+			(xy 198.755 146.05) (xy 203.835 146.05)
+		)
+		(stroke
+			(width 0)
+			(type solid)
+		)
+	)
+	(wire
+		(pts
 			(xy 239.395 34.925) (xy 241.935 34.925)
 		)
@@
 	(wire
 		(pts
+			(xy 187.325 149.225) (xy 189.23 149.225)
+		)
+		(stroke
+			(width 0)
+			(type default)
+		)
+	)
+	(wire
+		(pts
 			(xy 32.385 81.915) (xy 34.925 81.915)
 		)
@@
 	(wire
 		(pts
-			(xy 198.12 146.05) (xy 203.835 146.05)
+			(xy 198.12 146.05) (xy 198.755 146.05)
 		)
 		(stroke
@@
 			)
 		)
-		(property "MPN" "Generic C/2.2uF/C0G/25V/0603"
+		(property "MPN" "Generic C/2.2uF/X5R/25V/0603"
 			(at 67.945 53.975 0)
 			(effects
@@
 			)
 		)
-		(property "MPN" "Generic C/2.2uF/C0G/25V/0603"
+		(property "MPN" "Generic C/2.2uF/X5R/25V/0603"
 			(at 57.785 53.975 0)
 			(effects
@@
 			)
 		)
-		(property "MPN" "Generic C/1uF/C0G/25V/0603"
+		(property "MPN" "Generic C/1uF/X7R/25V/0603"
 			(at 228.6 152.4 0)
 			(effects
@@
 			)
 		)
-		(property "MPN" "Generic C/100nF/C0G/25V/0603"
+		(property "MPN" "Generic C/100nF/X7R/50V/0603"
 			(at 238.125 152.4 0)
 			(effects
@@
 			)
 		)
-		(property "MPN" "Generic C/100nF/C0G/25V/0603"
+		(property "MPN" "Generic C/100nF/X7R/50V/0603"
 			(at 151.13 107.95 0)
 			(effects
@@
 			)
 		)
-		(property "MPN" "Generic C/10nF/C0G/25V/0603"
+		(property "MPN" "Generic C/10nF/X7R/25V/0603"
 			(at 160.02 107.95 0)
 			(effects
@@
 			)
 		)
-		(property "MPN" "Generic C/100nF/C0G/25V/0603"
+		(property "MPN" "Generic C/100nF/X7R/50V/0603"
 			(at 170.18 107.95 0)
 			(effects
@@
 			)
 		)
-		(property "MPN" "Generic C/100nF/C0G/25V/0603"
+		(property "MPN" "Generic C/100nF/X7R/50V/0603"
 			(at 189.23 107.95 0)
 			(effects
@@
 			)
 		)
-		(property "MPN" "Generic C/10nF/C0G/25V/0603"
+		(property "MPN" "Generic C/10nF/X7R/25V/0603"
 			(at 198.12 107.95 0)
 			(effects
@@
 			)
 		)
-		(property "MPN" "Generic C/1uF/C0G/25V/0603"
+		(property "MPN" "Generic C/1uF/X7R/25V/0603"
 			(at 227.33 107.95 0)
 			(effects
@@
 			)
 		)
-		(property "MPN" "Generic C/100nF/C0G/25V/0603"
+		(property "MPN" "Generic C/100nF/X7R/50V/0603"
 			(at 187.325 77.47 0)
 			(effects
@@
 			)
 		)
-		(property "MPN" "Generic C/100nF/C0G/25V/0603"
+		(property "MPN" "Generic C/100nF/X7R/50V/0603"
 			(at 109.855 182.88 0)
 			(effects
@@
 			)
 		)
-		(property "MPN" "Generic C/100nF/C0G/25V/0603"
+		(property "MPN" "Generic C/100nF/X7R/50V/0603"
 			(at 140.335 182.88 0)
 			(effects
@@
 			)
 		)
-		(property "MPN" "Generic C/1uF/C0G/25V/0603"
+		(property "MPN" "Generic C/1uF/X7R/25V/0603"
 			(at 149.225 182.88 0)
 			(effects
@@
 		(in_bom yes)
 		(on_board yes)
-		(dnp no)
+		(dnp yes)
 		(fields_autoplaced yes)
 		(property "Reference" "JP201"
@@
 			)
 		)
-		(property "MPN" "Generic C/100nF/C0G/25V/0603"
+		(property "MPN" "Generic C/100nF/X7R/50V/0603"
 			(at 208.28 107.95 0)
 			(effects
@@
 	(symbol
 		(lib_id "Device:C_Small")
-		(at 182.245 151.13 0)
+		(at 182.245 156.845 0)
 		(unit 1)
 		(exclude_from_sim no)
@@
 		(dnp no)
 		(property "Reference" "C223"
-			(at 184.5818 149.9616 0)
+			(at 184.5818 155.6766 0)
 			(effects
 				(font
@@
 		)
 		(property "Value" "22u"
-			(at 184.5818 152.273 0)
+			(at 184.5818 157.988 0)
 			(effects
 				(font
@@
 		)
 		(property "Footprint" "Capacitor_SMD:C_1206_3216Metric"
-			(at 182.245 151.13 0)
+			(at 182.245 156.845 0)
 			(effects
 				(font
@@
 		)
 		(property "Datasheet" ""
-			(at 182.245 151.13 0)
+			(at 182.245 156.845 0)
 			(effects
 				(font
@@
 		)
 		(property "Description" ""
-			(at 182.245 151.13 0)
+			(at 182.245 156.845 0)
 			(effects
 				(font
@@
 		)
 		(property "MPN" "Generic C/22uF/X7R/10V/1206"
-			(at 182.245 151.13 0)
+			(at 182.245 156.845 0)
 			(effects
 				(font
@@
 			)
 		)
-		(property "MPN" "Generic C/100nF/C0G/25V/0603"
+		(property "MPN" "Generic C/100nF/X7R/50V/0603"
 			(at 273.685 152.4 0)
 			(effects
@@
 	)
 	(symbol
+		(lib_id "Device:R")
+		(at 193.04 149.225 270)
+		(unit 1)
+		(exclude_from_sim no)
+		(in_bom yes)
+		(on_board yes)
+		(dnp no)
+		(property "Reference" "R233"
+			(at 193.04 151.765 90)
+			(effects
+				(font
+					(size 1.27 1.27)
+				)
+			)
+		)
+		(property "Value" "0"
+			(at 193.04 149.225 90)
+			(effects
+				(font
+					(size 1.27 1.27)
+				)
+			)
+		)
+		(property "Footprint" "Resistor_SMD:R_0603_1608Metric"
+			(at 193.04 147.447 90)
+			(effects
+				(font
+					(size 1.27 1.27)
+				)
+				(hide yes)
+			)
+		)
+		(property "Datasheet" "~"
+			(at 193.04 149.225 0)
+			(effects
+				(font
+					(size 1.27 1.27)
+				)
+				(hide yes)
+			)
+		)
+		(property "Description" "Resistor"
+			(at 193.04 149.225 0)
+			(effects
+				(font
+					(size 1.27 1.27)
+				)
+				(hide yes)
+			)
+		)
+		(property "MPN" "Generic R/0R/0603"
+			(at 193.04 149.225 0)
+			(effects
+				(font
+					(size 1.27 1.27)
+				)
+				(hide yes)
+			)
+		)
+		(pin "2"
+		)
+		(pin "1"
+		)
+		(instances
+			(project "Module17-Mainboard"
+				(path "/59592280-3207-432b-a891-cd517ec5cf12/00000000-0000-0000-0000-0000612c95ef"
+					(reference "R233")
+					(unit 1)
+				)
+			)
+		)
+	)
+	(symbol
 		(lib_id "Device:R_Small")
 		(at 81.915 149.86 0)
@@
 	(symbol
 		(lib_id "power:GND")
-		(at 182.245 153.67 0)
+		(at 182.245 159.385 0)
 		(unit 1)
 		(exclude_from_sim no)
@@
 		(dnp no)
 		(property "Reference" "#PWR0264"
-			(at 182.245 160.02 0)
+			(at 182.245 165.735 0)
 			(effects
 				(font
@@
 		)
 		(property "Value" "GND"
-			(at 182.372 158.0642 0)
+			(at 182.372 163.7792 0)
 			(effects
 				(font
@@
 		)
 		(property "Footprint" ""
-			(at 182.245 153.67 0)
+			(at 182.245 159.385 0)
 			(effects
 				(font
@@
 		)
 		(property "Datasheet" ""
-			(at 182.245 153.67 0)
+			(at 182.245 159.385 0)
 			(effects
 				(font
@@
 		)
 		(property "Description" ""
-			(at 182.245 153.67 0)
+			(at 182.245 159.385 0)
 			(effects
 				(font
@@
 			)
 		)
-		(property "MPN" "Generic C/1uF/C0G/25V/0603"
+		(property "MPN" "Generic C/1uF/X7R/25V/0603"
 			(at 263.525 152.4 0)
 			(effects
@@
 			)
 		)
-		(property "MPN" "Generic C/100nF/C0G/25V/0603"
+		(property "MPN" "Generic C/100nF/X7R/50V/0603"
 			(at 141.605 134.62 0)
 			(effects
@@
 			)
 		)
-		(property "MPN" "Generic C/10nF/C0G/25V/0603"
+		(property "MPN" "Generic C/10nF/X7R/25V/0603"
 			(at 34.925 152.4 0)
 			(effects
@@
 			)
 		)
-		(property "MPN" "Generic C/10nF/C0G/25V/0603"
+		(property "MPN" "Generic C/10nF/X7R/25V/0603"
 			(at 179.07 107.95 0)
 			(effects
@@
 			)
 		)
-		(property "MPN" "Generic C/10nF/C0G/25V/0603"
+		(property "MPN" "Generic C/10nF/X7R/25V/0603"
 			(at 217.17 107.95 0)
 			(effects
@@
 			)
 		)
-		(property "MPN" "Generic C/10uF/C0G/25V/1210"
+		(property "MPN" "Generic C/10uF/X7R/25V/1210"
 			(at 107.315 151.13 0)
 			(effects

Commit message: Updated Mainboard PCB to revision 1.0
Other:
- company: M17Project -> M17 Project
Changed lines of the file:
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@@
 	(title_block
 		(title "Module17")
-		(date "2024-04-25")
-		(rev "Rev 0.99b")
-		(company "M17Project")
-		(comment 1 "Morgan ON4MOD")
+		(date "2024-06-19")
+		(rev "Rev 1.0")
+		(company "M17 Project")
+		(comment 1 "Morgan - ON4MOD")
 		(comment 2 "Mathis - DB9MAT")
 		(comment 3 "Wojciech - SP5WWP")
