File: hardware/HMI/Module17-HMI.kicad_pcb (KiCad board)
At the start: 4 copper layers, 97 x 80.9 mm, 59 parts, among them J1 Hirose FH12-26S-0.5SH(55), J3 Hirose FH12A-24S-0.5SH(55), Q1 MMBT3904, Q2 BSS84, SW9 CL-SB-22A-11T, U1 TPS61040DBV, U2 AP7375-33SA, U3 IQS211B00000000TS, U4 CAP1206-1-SL

Commit message: Added OSHWA certification mark
Parts:
- removed LOGO3: OSHW_logo, M17_logos:OSHW_logo_12.5x13mm
- added LOGO101: ~, OSHW_Certification_Mark:OSHW-Certification-Mark-Stacked_12x10mm_SilkMask, B.Cu at (211.4, 116.3)
Other:
- board text added: "Licensed under CERN-OHL-W v2"
